Commit message: rename pybullet part

File: pybullet_manipulator_gym/er_description/urdf/er6-730.urdf (robot description, URDF)
Before this commit: robot er6-730-mi, 9 links, 8 joints
Links:
- link base_link: mass None -> 4.0
- link ee_link: geometry collision box size=0.01 0.01 0.01
- link fifth_link: mass None -> 1.219
- link fourth_link: mass None -> 2.275
- link second_link: mass None -> 3.7
- link seventh_link: mass None -> 0.1879
- link sixth_link: mass None -> 1.219
- link third_link: mass None -> 8.393
Joints:
- joint base_fixed: origin xyz=0.0 0.0 0.0 rpy=0 0 3.14 -> xyz=0.0 0.0 0.0 rpy=0 0 0.0
